Commit message: made model urdf with leg

File: sawtooth_description/urdf/constants.xacro (robot description, xacro)
@@ -1,3 +1,19 @@
 <?xml version = "1.0"?>
 <robot xmlns:xacro="http://www.ros.org/wiki/xacro">
+    <!-- collision values -->
+    <!-- body -->
+    <xacro:property name="body_mass" value="0.700" />
+    <!-- body_mass is approx, change accordingly -->
+    <xacro:property name="body_length" value="0.160" />
+    <xacro:property name="body_width" value="0.253" />
+    <xacro:property name="body_height" value="0.050" />
+    <!-- hip -->
+    <xacro:property name="hip_mass" value="0.020" />
+    <xacro:property name="hip_radius" value="0.025" />
+    <xacro:property name="hip_length" value="0.050" />
+    <!-- femur -->
+    <xacro:property name="femur_mass" value="0.030" />
+    <xacro:property name="femur_length" value="0.015"/>
+    <xacro:property name="femur_width" value="0.100"/>
+    <xacro:property name="femur_height" value="0.100"/>
 </robot>

File: sawtooth_description/urdf/leg.xacro (robot description, xacro)
@@ -1,3 +1,70 @@
 <?xml version = "1.0"?>
 <robot xmlns:xacro="http://www.ros.org/wiki/xacro">
+    <xacro:macro name="leg" params="prefix">
+        <!-- hip link -->
+        <link name="${prefix}_hip">
+            <visual>
+                <origin xyz="0 0 0" rpy="${pi/2.0} 0 0" />
+                <geometry>
+                    <cylinder radius="${hip_radius}" length="${hip_length}" />
+                </geometry>
+                <material name="grey"/>
+            </visual>
+            <collision>
+                <origin xyz="0 0 0" rpy="0 0 0" />
+                <geometry>
+                    <cylinder radius="${hip_radius}" length="${hip_length}" />
+                </geometry>
+            </collision>
+            <!-- <inertial>
+                <mass value="${hip_mass}" />
+                <origin xyz="0 0 0" rpy="0 0 0"/>
+                inertia of cylinder
+                <interia ixx="${(hip_mass/12) * (3*hip_radius*hip_radius + hip_length*hip_length)}"    ixy="0.0"   ixz="0.0"
+                                    iyy="${(hip_mass/12) * (3*hip_radius*hip_radius + hip_length*hip_length)}"     iyz="0.0"
+                                                izz="${(hip_mass*hip_radius*hip_radius)/2}" />
+            </inertial> -->
+        </link>
+        <!-- femur link -->
+        <link name="${prefix}_femur">
+            <visual>
+                <origin xyz="-0.010 -0.010 -0.050" rpy="0 0 0"/>
+                <material name="black"/>
+                <geometry>
+                    <mesh filename="package://sawtooth_description/meshes/urdf_femur.stl" scale="1 1 1"/>
+                </geometry>
+            </visual>
+            <collision>
+                <origin xyz="0 0 0" rpy="0 0 0"/>
+                <geometry>
+                    <mesh filename="package://sawtooth_description/meshes/urdf_femur.stl" scale="1 1 1"/>
+                </geometry>
+            </collision>
+            <inertal>
+                <mass value="${femur_mass}"/>
+                <origin xyz="0 0 0" rpy="0 0 0"/>
+                <!-- inertia of box -->
+                <inertia
+                    ixx="${(femur_mass/12) * (femur_width * femur_width + femur_height * femur_height)}"  ixy="0.0"  ixz="0.0"
+                            iyy="${(femur_mass/12) * (femur_height * femur_height + femur_length * femur_length)}"   iyz="0.0"
+                                    izz="${(femur_mass/12) * (femur_width * femur_width + femur_length * femur_length)}"/>
+            </inertal>
+        </link>
+        <!-- Joints -->
+        <joint name="body_${prefix}_hip_joint" type="revolute">
+            <parent link="body" />
+            <child link="${prefix}_hip" />
+            <origin xyz="${body_length/3} ${body_width/3} ${body_height/2}" rpy="0 0 0" />
+            <axis xyz="0 1 0" />
+            <limit lower="-1.0" upper="1.0" effort="100" velocity="100" />
+        </joint>
+        <joint name="hip_femur_joint" type="revolute">
+            <parent link="${prefix}_hip" />
+            <child link="${prefix}_femur" />
+            <origin xyz="${hip_radius} 0 0" rpy="0 0 0" />
+            <axis xyz="1 0 0" />
+            <limit lower="-1.0" upper="1.0" effort="100" velocity="100" />
+        </joint>
+<!-- ${body_width/6} -->
+    </xacro:macro>
 </robot>

File: sawtooth_description/urdf/materials.xacro (robot description, xacro)
@@ -12,5 +12,5 @@
     </material>
     <material name="grey">
-        <color rgba="0.2 0.2 0.2 0.0"/>
+        <color rgba="0.2 0.2 0.2 1.0"/>
     </material>
     <material name="silver">
@@ -29,3 +29,6 @@
         <color rgba="1.0 1.0 1.0 1.0"/>
     </material>
+    <material name="yellow">
+        <color rgba="1.0 1.0 0.0 1.0"/>
+    </material>
 </robot>

File: sawtooth_description/urdf/sawtooth_robot.xacro (robot description, xacro)
@@ -5,5 +5,44 @@
     <xacro:include filename="$(find sawtooth_description)/urdf/constants.xacro" />
     <xacro:include filename="$(find sawtooth_description)/urdf/materials.xacro" />
+    <xacro:include filename="$(find sawtooth_description)/urdf/leg.xacro" />
+    <!-- Location of leg(motor) joints are for simulation only-->
     <!-- links -->
+    <!-- base_link = dummy (mandetory) link. It acts as the root reference for other links. -->
+    <link name="base_link"/>
+    <link name="body">
+        <visual>
+            <origin xyz="0.0 0.0 0.0" rpy="0.0 0.0 0.0"/>
+            <geometry>
+                <mesh filename="package://sawtooth_description/meshes/urdf_base.stl" scale="1 1 1"/>
+            </geometry>
+            <material name="orange"/>
+        </visual>
+        <collision>
+            <origin xyz="0.0 0.0 0.0" rpy="0.0 0.0 0.0"/>
+            <geometry>
+                <mesh filename="package://sawtooth_description/meshes/urdf_base.stl" scale="1 1 1"/>
+            </geometry>
+        </collision>
+        <inertial>
+            <mass value="${body_mass}"/>
+            <origin xyz="0 0 0.025" rpy="0 0 0"/>
+            <!-- inertia of box -->
+            <inertia
+                ixx="${(body_mass/12) * (body_width * body_width + body_height * body_height)}"  ixy="0.0"  ixz="0.0"
+                        iyy="${(body_mass/12) * (body_height * body_height + body_length * body_length)}"   iyz="0.0"
+                                izz="${(body_mass/12) * (body_width * body_width + body_length * body_length)}"/>
+        </inertial>
+        <!-- you cannot nest ${...} inside another ${...}, no need to wrap each variable with ${} again — just use them like normal variables inside the arithmetic. -->
+    </link>
+    <xacro:leg prefix="front_left"/>
     <!-- joints -->
+    <joint name="baselink_body_joint" type="fixed">
+        <parent link="base_link" />
+        <child link="body" />
+        <origin xyz="0 0 0" rpy="0 0 0" />
+    </joint>
 </robot>
+<!-- for this project:
+    length = x
+    width = y
+    height = z -->

Commit message: urdf completed

File: sawtooth_description/urdf/constants.xacro (robot description, xacro)
@@ -17,3 +17,14 @@
     <xacro:property name="femur_width" value="0.100"/>
     <xacro:property name="femur_height" value="0.100"/>
+    <!-- tibia -->
+    <xacro:property name="tibia_mass" value="0.014" />
+    <xacro:property name="tibia_length" value="0.008"/>
+    <xacro:property name="tibia_width" value="0.112"/>
+    <xacro:property name="tibia_height" value="0.112"/>
+    <!-- offset values -->
+    <xacro:property name="femur_joint_offset_x" value="0.010"/>
+    <xacro:property name="femur_visual_offset_x" value="0.010"/>
+    <xacro:property name="Rfemur_visual_offset_x" value="0.030"/>
+    <xacro:property name="femur_visual_offset_y" value="0.010"/>
+    <xacro:property name="femur_visual_offset_z" value="0.050"/>
 </robot>

File: sawtooth_description/urdf/leg.xacro (robot description, xacro)
@@ -1,5 +1,5 @@
 <?xml version = "1.0"?>
 <robot xmlns:xacro="http://www.ros.org/wiki/xacro">
-    <xacro:macro name="leg" params="prefix">
+    <xacro:macro name="leg" params="prefix front_rear side">
         <!-- hip link -->
         <link name="${prefix}_hip">
@@ -12,23 +12,30 @@
             </visual>
             <collision>
-                <origin xyz="0 0 0" rpy="0 0 0" />
+                <origin xyz="0 0 0" rpy="${pi/2.0} 0 0" />
                 <geometry>
                     <cylinder radius="${hip_radius}" length="${hip_length}" />
                 </geometry>
             </collision>
-            <!-- <inertial>
+            <inertial>
                 <mass value="${hip_mass}" />
                 <origin xyz="0 0 0" rpy="0 0 0"/>
-                inertia of cylinder
-                <interia ixx="${(hip_mass/12) * (3*hip_radius*hip_radius + hip_length*hip_length)}"    ixy="0.0"   ixz="0.0"
-                                    iyy="${(hip_mass/12) * (3*hip_radius*hip_radius + hip_length*hip_length)}"     iyz="0.0"
-                                                izz="${(hip_mass*hip_radius*hip_radius)/2}" />
-            </inertial> -->
+                <!-- inertia of cylinder -->
+                <inertia ixx="${(hip_mass/12) * (3 * hip_radius * hip_radius + hip_length * hip_length)}"    ixy="0.0"   ixz="0.0"
+                                    iyy="${(hip_mass/12) * (3 * hip_radius * hip_radius + hip_length * hip_length)}"     iyz="0.0"
+                                                izz="${(hip_mass * hip_radius * hip_radius)/2}" />
+            </inertial>
         </link>
         <!-- femur link -->
         <link name="${prefix}_femur">
             <visual>
-                <origin xyz="-0.010 -0.010 -0.050" rpy="0 0 0"/>
-                <material name="black"/>
+                <!-- if left -->
+                <xacro:if value="${(side == 1)}">
+                    <origin xyz="${-femur_visual_offset_x} ${-femur_visual_offset_y} ${-femur_visual_offset_z}" rpy="0 0 0"/>
+                </xacro:if>
+                <!-- if right -->
+                <xacro:if value="${side == -1}">
+                    <origin xyz="${-Rfemur_visual_offset_x} ${-femur_visual_offset_y} ${-femur_visual_offset_z}" rpy="0 0 0"/>
+                </xacro:if>
+                <material name="white"/>
                 <geometry>
                     <mesh filename="package://sawtooth_description/meshes/urdf_femur.stl" scale="1 1 1"/>
@@ -36,10 +43,10 @@
             </visual>
             <collision>
-                <origin xyz="0 0 0" rpy="0 0 0"/>
+                <origin xyz="-0.010 -0.010 -0.050" rpy="0 0 0"/>
                 <geometry>
                     <mesh filename="package://sawtooth_description/meshes/urdf_femur.stl" scale="1 1 1"/>
                 </geometry>
             </collision>
-            <inertal>
+            <inertial>
                 <mass value="${femur_mass}"/>
                 <origin xyz="0 0 0" rpy="0 0 0"/>
@@ -49,5 +56,31 @@
                             iyy="${(femur_mass/12) * (femur_height * femur_height + femur_length * femur_length)}"   iyz="0.0"
                                     izz="${(femur_mass/12) * (femur_width * femur_width + femur_length * femur_length)}"/>
-            </inertal>
+            </inertial>
+        </link>
+        <link name="${prefix}_tibia">
+            <visual>
+                <origin xyz="-0.02 -0.088 0.025" rpy="0 0 0" />
+                <geometry>
+                    <mesh filename="package://sawtooth_description/meshes/urdf_tibia.stl" scale="1 1 1" />
+                </geometry>
+                <material name="black"/>
+            </visual>
+            <collision>
+                <origin xyz="-0.02 -0.088 0.025" rpy="0 0 0" />
+                <geometry>
+                    <mesh filename="package://sawtooth_description/meshes/urdf_tibia.stl" scale="1 1 1" />
+                </geometry>
+            </collision>
+            <inertial>
+                <mass value="${tibia_mass}" />
+                <origin xyz="0 0 0" />
+                <!-- inertia of box -->
+                <inertia ixx="${(tibia_mass/12) * (tibia_width * tibia_width + tibia_height * tibia_height)}"
+                         ixy="0.0"
+                         ixz="0.0"
+                         iyy="${(tibia_mass/12) * (tibia_height * tibia_height + tibia_length * tibia_length)}"
+                         iyz="0.0"
+                         izz="${(tibia_mass/12) * (tibia_width * tibia_width + tibia_length * tibia_length)}" />
+            </inertial>
         </link>
         <!-- Joints -->
@@ -55,16 +88,22 @@
             <parent link="body" />
             <child link="${prefix}_hip" />
-            <origin xyz="${body_length/3} ${body_width/3} ${body_height/2}" rpy="0 0 0" />
+            <origin xyz="${side*body_length/3} ${front_rear*body_width/3} ${body_height/2}" rpy="0 0 0" />
             <axis xyz="0 1 0" />
             <limit lower="-1.0" upper="1.0" effort="100" velocity="100" />
         </joint>
-        <joint name="hip_femur_joint" type="revolute">
+        <joint name="${prefix}_hip_femur_joint" type="revolute">
             <parent link="${prefix}_hip" />
             <child link="${prefix}_femur" />
-            <origin xyz="${hip_radius} 0 0" rpy="0 0 0" />
+            <origin xyz="${side*hip_radius} 0 0" rpy="0 0 0" />
             <axis xyz="1 0 0" />
             <limit lower="-1.0" upper="1.0" effort="100" velocity="100" />
         </joint>
-<!-- ${body_width/6} -->
+        <joint name="${prefix}_femur_tibia_joint" type="revolute">
+            <parent link="${prefix}_femur" />
+            <child link="${prefix}_tibia" />
+            <origin xyz="${side*femur_joint_offset_x} ${femur_width-0.022} ${-femur_height+0.025}" rpy="0 0 0" />
+            <axis xyz="1 0 0" />
+            <limit lower="-1.0" upper="1.0" effort="100" velocity="100" />
+        </joint>
     </xacro:macro>
 </robot>

File: sawtooth_description/urdf/sawtooth_robot.xacro (robot description, xacro)
@@ -35,5 +35,11 @@
         <!-- you cannot nest ${...} inside another ${...}, no need to wrap each variable with ${} again — just use them like normal variables inside the arithmetic. -->
     </link>
-    <xacro:leg prefix="front_left"/>
+    <!--prefix → leg name (e.g., FL, FR, HL, HR).
+        side → 1 (left) or -1 (right).
+        front_rear → 1 (rear) or -1 (front). -->
+    <xacro:leg prefix="FL" front_rear="-1" side="1"/>
+    <xacro:leg prefix="FR" front_rear="-1" side="-1"/>
+    <xacro:leg prefix="RL" front_rear="1" side="1"/>
+    <xacro:leg prefix="RR" front_rear="1" side="-1"/>
     <!-- joints -->
     <joint name="baselink_body_joint" type="fixed">
@@ -43,6 +49,3 @@
     </joint>
 </robot>
-<!-- for this project:
-    length = x
-    width = y
-    height = z -->
+<!-- for this project: x = length | y = width | z = height -->

Commit message: spawned in gazebo

File: sawtooth_description/urdf/constants.xacro (robot description, xacro)
@@ -28,3 +28,6 @@
     <xacro:property name="femur_visual_offset_y" value="0.010"/>
     <xacro:property name="femur_visual_offset_z" value="0.050"/>
+    <xacro:property name="tibia_visual_offset_x" value="0.02"/>
+    <xacro:property name="tibia_visual_offset_y" value="0.088"/>
+    <xacro:property name="tibia_visual_offset_z" value="0.025"/>
 </robot>

File: sawtooth_description/urdf/leg.xacro (robot description, xacro)
@@ -21,7 +21,10 @@
                 <origin xyz="0 0 0" rpy="0 0 0"/>
                 <!-- inertia of cylinder -->
-                <inertia ixx="${(hip_mass/12) * (3 * hip_radius * hip_radius + hip_length * hip_length)}"    ixy="0.0"   ixz="0.0"
-                                    iyy="${(hip_mass/12) * (3 * hip_radius * hip_radius + hip_length * hip_length)}"     iyz="0.0"
-                                                izz="${(hip_mass * hip_radius * hip_radius)/2}" />
+                <inertia ixx="${(hip_mass/12) * (3 * hip_radius * hip_radius + hip_length * hip_length)}"
+                         ixy="0.0"
+                         ixz="0.0"
+                         iyy="${(hip_mass/12) * (3 * hip_radius * hip_radius + hip_length * hip_length)}"
+                         iyz="0.0"
+                         izz="${(hip_mass * hip_radius * hip_radius)/2}" />
             </inertial>
         </link>
@@ -31,9 +34,13 @@
                 <!-- if left -->
                 <xacro:if value="${(side == 1)}">
-                    <origin xyz="${-femur_visual_offset_x} ${-femur_visual_offset_y} ${-femur_visual_offset_z}" rpy="0 0 0"/>
+                    <origin xyz="${-femur_visual_offset_x}
+                                 ${-femur_visual_offset_y}
+                                 ${-femur_visual_offset_z}" rpy="0 0 0"/>
                 </xacro:if>
                 <!-- if right -->
                 <xacro:if value="${side == -1}">
-                    <origin xyz="${-Rfemur_visual_offset_x} ${-femur_visual_offset_y} ${-femur_visual_offset_z}" rpy="0 0 0"/>
+                    <origin xyz="${-Rfemur_visual_offset_x}
+                                 ${-femur_visual_offset_y}
+                                 ${-femur_visual_offset_z}" rpy="0 0 0"/>
                 </xacro:if>
                 <material name="white"/>
@@ -43,5 +50,16 @@
             </visual>
             <collision>
-                <origin xyz="-0.010 -0.010 -0.050" rpy="0 0 0"/>
+                <!-- if left -->
+                <xacro:if value="${(side == 1)}">
+                    <origin xyz="${-femur_visual_offset_x}
+                                 ${-femur_visual_offset_y}
+                                 ${-femur_visual_offset_z}" rpy="0 0 0"/>
+                </xacro:if>
+                <!-- if right -->
+                <xacro:if value="${side == -1}">
+                    <origin xyz="${-Rfemur_visual_offset_x}
+                                 ${-femur_visual_offset_y}
+                                 ${-femur_visual_offset_z}" rpy="0 0 0"/>
+                </xacro:if>
                 <geometry>
                     <mesh filename="package://sawtooth_description/meshes/urdf_femur.stl" scale="1 1 1"/>
@@ -53,12 +71,17 @@
                 <!-- inertia of box -->
                 <inertia
-                    ixx="${(femur_mass/12) * (femur_width * femur_width + femur_height * femur_height)}"  ixy="0.0"  ixz="0.0"
-                            iyy="${(femur_mass/12) * (femur_height * femur_height + femur_length * femur_length)}"   iyz="0.0"
-                                    izz="${(femur_mass/12) * (femur_width * femur_width + femur_length * femur_length)}"/>
+                    ixx="${(femur_mass/12) * (femur_width * femur_width + femur_height * femur_height)}"
+                    ixy="0.0"
+                    ixz="0.0"
+                    iyy="${(femur_mass/12) * (femur_height * femur_height + femur_length * femur_length)}"
+                    iyz="0.0"
+                    izz="${(femur_mass/12) * (femur_width * femur_width + femur_length * femur_length)}"/>
             </inertial>
         </link>
         <link name="${prefix}_tibia">
             <visual>
-                <origin xyz="-0.02 -0.088 0.025" rpy="0 0 0" />
+                <origin xyz="${-tibia_visual_offset_x}
+                             ${-tibia_visual_offset_y}
+                             ${tibia_visual_offset_z}" rpy="0 0 0" />
                 <geometry>
                     <mesh filename="package://sawtooth_description/meshes/urdf_tibia.stl" scale="1 1 1" />
@@ -67,5 +90,7 @@
             </visual>
             <collision>
-                <origin xyz="-0.02 -0.088 0.025" rpy="0 0 0" />
+                <origin xyz="${-tibia_visual_offset_x}
+                             ${-tibia_visual_offset_y}
+                             ${tibia_visual_offset_z}" rpy="0 0 0" />
                 <geometry>
                     <mesh filename="package://sawtooth_description/meshes/urdf_tibia.stl" scale="1 1 1" />
@@ -88,5 +113,7 @@
             <parent link="body" />
             <child link="${prefix}_hip" />
-            <origin xyz="${side*body_length/3} ${front_rear*body_width/3} ${body_height/2}" rpy="0 0 0" />
+            <origin xyz="${side*body_length/3}
+                         ${front_rear*body_width/3}
+                         ${body_height/2}" rpy="0 0 0" />
             <axis xyz="0 1 0" />
             <limit lower="-1.0" upper="1.0" effort="100" velocity="100" />

File: sawtooth_description/urdf/sawtooth_gazebo.xacro (robot description, xacro)
@@ -2,3 +2,9 @@
 <robot xmlns:xacro="http://www.ros.org/wiki/xacro">
     <!-- Gazebo Sim Plug-ins -->
+    <!-- https://github.com/gazebosim/gz-sim/tree/gz-sim9/src/systems -->
+    <!-- to simulate (fake) motor encoders -->
+    <gazebo>
+        <plugin
+            filename="gz-sim-joint-state-publisher-system"
+            name="gz::sim::systems::JointStatePublisher">
 </robot>

File: sawtooth_description/urdf/sawtooth_robot.xacro (robot description, xacro)
@@ -49,3 +49,4 @@
     </joint>
 </robot>
-<!-- for this project: x = length | y = width | z = height -->
+<!-- for this project -> x => length | y => width | z => height -->
+<!-- don't use colcons anywhere in urdf/xacro file in comments, bcz xml parser don't allow -->
